Commit message: fix errors for conda env

File: launch/ego_racecar.xacro (robot description, xacro)
@@ -74,7 +74,8 @@
   </joint>
   <link name="${car_name}/front_left_hinge"/>
-  <joint name="front_left_hinge_to_wheel" type="continuous">
+  <joint name="front_left_hinge_to_wheel" type="fixed">
     <parent link="${car_name}/front_left_hinge"/>
     <child link="${car_name}/front_left_wheel"/>
+    <origin xyz="0 0 0"/>
   </joint>
   <link name="${car_name}/front_left_wheel">
@@ -93,7 +94,8 @@
   </joint>
   <link name="${car_name}/front_right_hinge"/>
-  <joint name="front_right_hinge_to_wheel" type="continuous">
+  <joint name="front_right_hinge_to_wheel" type="fixed">
     <parent link="${car_name}/front_right_hinge"/>
     <child link="${car_name}/front_right_wheel"/>
+    <origin xyz="0 0 0"/>
   </joint>
   <link name="${car_name}/front_right_wheel">
